Commit message: robko urdf model with 3 decks

File: src/robko18_description/urdf/robko18.xacro (robot description, xacro)
@@ -1,13 +1,100 @@
 <?xml version='1.0'?>
-<robot name="myrobot" xmlns:xacro="http://www.ros.org/wiki/xacro">
-  <xacro:property name="cameraSize" value="0.05"/>
-  <xacro:property name="cameraMass" value="0.1"/>
+<robot name="robko18" xmlns:xacro="http://www.ros.org/wiki/xacro">
   <xacro:include filename="$(find robko18_description)/urdf/robko18.gazebo" />
   <xacro:include filename="$(find robko18_description)/urdf/materials.xacro" />
   <xacro:include filename="$(find robko18_description)/urdf/macros.xacro" />
-  <link name='chassis'>
+  <!-- ####### generic constants ##### -->
+  <!--All units in m-kg-s-radians unit system -->
+  <xacro:property name="M_PI" value="3.1415926535897931" />
+  <xacro:property name="M_PI_2" value="1.570796327" />
+  <xacro:property name="DEG_TO_RAD" value="0.017453293" />
+  <xacro:property name="SCALE_in_m" value="0.0254"/> <!--inches to meters-->
+  <xacro:property name="SCALE_mm_m" value="0.001"/> <!--milimeters to meters-->
+   <!-- robot constants -->
+    <!-- Main body radius and height -->
+    <!--Base Plate Dimensions: 0.375" (0.95 cm) thick x 17.75" (45.09 cm) diameter
+Double Battery Shelf Dimensions: 0.375" (0.95 cm) thick x 7.0" (17.78 cm) x 13.25" ( 11.43 x 33.66 cm)
+Battery Containment Area Dimensions: 2.625" x 8.00" x 6.75"
+Weight = 3.85 lbs (1.75 kg)
+The Arlo top deck adds 5.375" (13.65 cm) of height when used with the Arlo Base Kit
+Overall height is 5.375 inches ( 13.65cm)
+Weight = 3.5 lbs (1.59 kg) per assembly
+Dimensions: 17.375 inches (44.13 cm) diameter x .375 inches (.95 cm) thick
+-->  second_deck
+  <!-- base_link - Base Plate/Deck Cylinder base   -->
+  <xacro:property name="base_from_base_frame_Z_offset" value="0.10"/>
+  <xacro:property name="base_height" value="${0.375*SCALE_in_m}" />
+  <xacro:property name="base_radius" value="${17.75*SCALE_in_m}" />
+  <!-- in kg weight with the battery holder plate bellow -->
+  <xacro:property name="base_mass" value="1.75" />
+   <!-- distance between the robot origin and the bottom of the base plate along the z axis (robot up) -->
+  <xacro:property name="BASE_PLATE_FROM_BASE_FRAME_Z_OFFSET" value="${0.10+(base_height/2)}" /> <!-- meters -->
+ <!-- second_deck - Base Plate/Deck Cylinder base   -->
+  <xacro:property name="second_deck_from_base_link_Z_offset" value="0.145"/>
+  <xacro:property name="second_deck_height" value="${0.375*SCALE_in_m}" />
+  <xacro:property name="second_deck_radius" value="${17.75*SCALE_in_m}" />
+  <xacro:property name="second_deck_mass" value="1.5" />   <!-- in kg -->
+  <!-- third_deck - Base Plate/Deck Cylinder base   -->
+  <xacro:property name="third_deck_from_base_link_Z_offset" value="0.145"/>
+  <xacro:property name="third_deck_height" value="${0.375*SCALE_in_m}" />
+  <xacro:property name="third_deck_radius" value="${17.75*SCALE_in_m}" />
+  <xacro:property name="third_deck_mass" value="1.5" />   <!-- in kg -->
+  <!-- Wheels -->
+  <xacro:property name="wheel_diameter" value="${6*SCALE_in_m}"/>
+  <xacro:property name="wheel_radius" value="${wheel_diameter/2}"/>
+  <xacro:property name="wheel_width" value="0.03"/><!--set to tyre width-->
+  <xacro:property name="wheel_mass" value="0.6" /> --> <!-- ???? in kg-->
+  <xacro:property name="base_x_origin_to_wheel_origin" value="0.0" />
+  <xacro:property name="base_y_origin_to_wheel_origin" value="0.2" />
+    <!--<xacro:property name="base_y_origin_to_wheel_origin" value="0.19" />-->
+  <xacro:property name="base_z_origin_to_wheel_origin" value="${BASE_PLATE_FROM_BASE_FRAME_Z_OFFSET - wheel_radius}" />
+  <!-- caster wheel offsets from base origin -->
+  <xacro:property name="caster_X_offset_from_base_link" value="0.17"/>
+  <!-- caster wheel radius and height -->
+  <!-- caster wheel mass -->
+  <xacro:property name="caster_box_mass" value="0.15" /> <!-- in kg-->
+  <xacro:property name="caster_box_height" value="0.05" />
+  <xacro:property name="caster_box_width" value="0.05" />
+  <xacro:property name="caster_box_lenght" value="0.05" />
+  <xacro:property name="caster_sphere_mass" value="0.15" /> <!-- in kg-->
+  <xacro:property name="caster_sphere_diameter" value="0.05" />
+  <xacro:property name="caster_sphere_radius" value="${caster_sphere_diameter/2}" />
+  <!-- SENSORS -->
+  <!-- Hokuyo Laser scanner -->
+  <xacro:property name="hokuyo_size" value="0.05" />
+    <!-- camera -->
+  <xacro:property name="cameraSize" value="0.05"/>
+  <xacro:property name="cameraMass" value="0.1"/>
+ <!-- base_footprint is a fictitious link(frame) that is on the ground right below base_link origin -->
+ <!--<link name="base_footprint"/>-->
+  <link name="base_footprint">
+    <inertial>
+      <mass value="0.0001"/>
+      <origin xyz="0 0 0"/>
+      <inertia ixx="0.0001" ixy="0.0" ixz="0.0" iyy="0.0001" iyz="0.0" izz="0.0001"/>
+    </inertial>
+    <visual>
+      <origin rpy="0 0 0" xyz="0 0 0"/>
+      <geometry>
+        <box size="0.001 0.001 0.001"/>
+      </geometry>
+      <material name="red"/>
+    </visual>
+  </link>
+  <gazebo reference="base_footprint">
+    <turnGravityOff>false</turnGravityOff>
+  </gazebo>
+  <!-- JOINT BASE_LINK TO BASE_FRAME-->
+  <joint name="base_footprint_base_link_joint" type="fixed">
+    <origin rpy="0 0 0" xyz="0 0 ${base_from_base_frame_Z_offset}"/>
+    <parent link="base_footprint"/>
+    <child link="base_link"/>
+  </joint>
+  <!-- BASE-LINK -->
+  <!--Center on the bottom side of the base plate of the robot-->
+  <link name='base_link'>
     <pose>0 0 0.1 0 0 0</pose>
     <inertial>
-      <mass value="15.0"/>
+      <mass value="${base_mass}"/>
       <origin xyz="0.0 0 0.1" rpy=" 0 0 0"/>
       <inertia
@@ -19,64 +106,21 @@
     <collision name='collision'>
       <geometry>
-        <box size=".4 .2 .1"/>
-      </geometry>
-    </collision>
-    <visual name='chassis_visual'>
-      <origin xyz="0 0 0" rpy=" 0 0 0"/>
-      <geometry>
-        <box size=".4 .2 .1"/>
-      </geometry>
-    </visual>
-    <collision name='caster_collision'>
-      <origin xyz="-0.15 0 -0.05" rpy=" 0 0 0"/>
-      <geometry>
-        <sphere radius="0.05"/>
-      </geometry>
-      <surface>
-        <friction>
-          <ode>
-            <mu>0</mu>
-            <mu2>0</mu2>
-            <slip1>1.0</slip1>
-            <slip2>1.0</slip2>
-          </ode>
-        </friction>
-      </surface>
-    </collision>
-    <visual name='caster_visual'>
-      <origin xyz="-0.15 0 -0.05" rpy=" 0 0 0"/>
-      <geometry>
-        <sphere radius="0.05"/>
-      </geometry>
-    </visual>
-    <collision name='caster_front_collision'>
-      <origin xyz="0.15 0 -0.05" rpy=" 0 0 0"/>
-      <geometry>
-        <sphere radius="0.05"/>
-      </geometry>
-      <surface>
-        <friction>
-          <ode>
-            <mu>0</mu>
-            <mu2>0</mu2>
-            <slip1>1.0</slip1>
-            <slip2>1.0</slip2>
-          </ode>
-        </friction>
-      </surface>
-    </collision>
-    <visual name='caster_front_visual'>
-      <origin xyz="0.15 0 -0.05" rpy=" 0 0 0"/>
-      <geometry>
-        <sphere radius="0.05"/>
-      </geometry>
+       <cylinder radius="${base_radius}" length="${base_height}"/>
+      </geometry>
+    </collision>
+    <visual name='base_visual'>
+      <origin xyz="0 0 0" rpy="${M_PI_2} 0 ${M_PI_2}"/>
+      <geometry>
+        <!--<cylinder radius="${base_radius}" length="${base_height}"/>-->
+        <mesh filename="$(find robko18_description)/meshes/ArloBottomplateTST.dae" scale="0.001 0.001 0.001"/>
+      </geometry>
+      <material name="orange"/>
     </visual>
   </link>
   <link name="left_wheel">
-    <!--origin xyz="0.1 0.13 0.1" rpy="0 1.5707 1.5707"/-->
-    <collision name="collision">
-      <origin xyz="0 0 0" rpy="0 1.5707 1.5707"/>
-      <geometry>
-        <cylinder radius="0.1" length="0.05"/>
+    <collision name="collision">
+      <origin xyz="0 0 0" rpy="0 1.5707 1.5707"/>
+      <geometry>
+        <cylinder radius="${wheel_radius}" length="${wheel_width}"/>
       </geometry>
     </collision>
@@ -84,5 +128,5 @@
       <origin xyz="0 0 0" rpy="0 1.5707 1.5707"/>
       <geometry>
-        <cylinder radius="0.1" length="0.05"/>
+        <cylinder radius="${wheel_radius}" length="${wheel_width}"/>
       </geometry>
     </visual>
@@ -97,9 +141,8 @@
   </link>
   <link name="right_wheel">
-    <!--origin xyz="0.1 -0.13 0.1" rpy="0 1.5707 1.5707"/-->
-    <collision name="collision">
-      <origin xyz="0 0 0" rpy="0 1.5707 1.5707"/>
-      <geometry>
-        <cylinder radius="0.1" length="0.05"/>
+    <collision name="collision">
+      <origin xyz="0 0 0" rpy="0 1.5707 1.5707"/>
+      <geometry>
+        <cylinder radius="${wheel_radius}" length="${wheel_width}"/>
       </geometry>
     </collision>
@@ -107,5 +150,5 @@
       <origin xyz="0 0 0" rpy="0 1.5707 1.5707"/>
       <geometry>
-        <cylinder radius="0.1" length="0.05"/>
+        <cylinder radius="${wheel_radius}" length="${wheel_width}"/>
       </geometry>
     </visual>
@@ -120,8 +163,8 @@
   </link>
   <joint type="continuous" name="left_wheel_hinge">
-    <origin xyz="0 0.15 0" rpy="0 0 0"/>
-    <!--origin xyz="0.1 0.13 0" rpy="0 1.5707 1.5707"/-->
+    <origin xyz="0 ${base_y_origin_to_wheel_origin} -${base_z_origin_to_wheel_origin}" rpy="0 0 0"/>
+        <!--<origin xyz="0 0.19 -${0.10 - 0.0231}" rpy="0 0 0"/>-->
     <child link="left_wheel"/>
-    <parent link="chassis"/>
+    <parent link="base_link"/>
     <axis xyz="0 1 0" rpy="0 0 0"/>
     <limit effort="10000" velocity="1000"/>
@@ -129,12 +172,204 @@
   </joint>
   <joint type="continuous" name="right_wheel_hinge">
-    <origin xyz="0 -0.15 0" rpy="0 0 0"/>
-    <!--origin xyz="0.1 -0.13 0" rpy="0 1.5707 1.5707"/-->
+    <origin xyz="0 -${base_y_origin_to_wheel_origin} -${base_z_origin_to_wheel_origin}" rpy="0 0 0"/>
+    <!--<origin xyz="0 -0.19 -0.0231" rpy="0 0 0"/>-->
     <child link="right_wheel"/>
-    <parent link="chassis"/>
+    <parent link="base_link"/>
     <axis xyz="0 1 0" rpy="0 0 0"/>
     <limit effort="10000" velocity="1000"/>
     <joint_properties damping="1.0" friction="1.0"/>
   </joint>
+<!--###########caster front #############################-->
+  <link name="caster_box_front">
+    <collision name="collision">
+      <origin xyz="0 0 0" rpy="0 0 0"/>
+      <geometry>
+        <box size="${caster_box_width} ${caster_box_height} ${caster_box_lenght}"/>
+      </geometry>
+    </collision>
+    <visual name="caster_box_front_visual">
+      <origin xyz="0 0 0" rpy="0 0 0"/>
+      <geometry>
+        <box size="${caster_box_width} ${caster_box_height} ${caster_box_lenght}"/>
+      </geometry>
+    </visual>
+    <inertial>
+      <origin xyz="0 0 0" rpy="0 0 0"/>
+      <mass value="0.15"/>
+      <inertia
+        ixx=".1" ixy="0.0" ixz="0.0"
+        iyy=".1" iyz="0.0"
+        izz=".1"/>
+    </inertial>
+  </link>
+    <!-- JOINT caster_box_front TO base_link-->
+  <joint name="base_caster_box_front_joint" type="fixed">
+  <!-- NB: Z goes to - as we are below bottom deck(base)-->
+    <origin rpy="0 0 0" xyz="${caster_X_offset_from_base_link+caster_box_lenght/2} 0 -${caster_box_height/2+base_height/2}"/>
+    <parent link="base_link"/>
+    <child link="caster_box_front"/>
+  </joint>
+     <!--*****************************-->
+    <link name="caster_sphere_front">
+    <collision name="collision">
+      <origin xyz="0 0 0" rpy="0 0 0"/>
+      <geometry>
+        <sphere radius="${caster_sphere_radius}"/>
+      </geometry>
+    </collision>
+    <visual name="caster_sphere_front_visual">
+      <origin xyz="0 0 0" rpy="0 0 0"/>
+      <geometry>
+        <sphere radius="${caster_sphere_radius}"/>
+      </geometry>
+    </visual>
+    <inertial>
+      <origin xyz="0 0 0" rpy="0 0 0"/>
+      <mass value="0.15"/>
+      <inertia
+        ixx=".1" ixy="0.0" ixz="0.0"
+        iyy=".1" iyz="0.0"
+        izz=".1"/>
+    </inertial>
+  </link>
+    <!-- JOINT caster_sphere_front TO caster_box_front-->
+  <joint name="caster_box_front_caster_sphere_front_joint" type="fixed">
+  <!-- NB: Z goes to - as we are below bottom deck(base)-->
+    <origin rpy="0 0 0" xyz="0 0 -${caster_box_lenght/2+caster_sphere_radius}"/>
+    <parent link="caster_box_front"/>
+    <child link="caster_sphere_front"/>
+  </joint>
+<!--########################################-->
+<!--###########caster back #############################-->
+  <link name="caster_box_back">
+    <collision name="collision">
+      <origin xyz="0 0 0" rpy="0 0 0"/>
+      <geometry>
+        <box size="${caster_box_width} ${caster_box_height} ${caster_box_lenght}"/>
+      </geometry>
+    </collision>
+    <visual name="caster_box_back_visual">
+      <origin xyz="0 0 0" rpy="0 0 0"/>
+      <geometry>
+        <box size="${caster_box_width} ${caster_box_height} ${caster_box_lenght}"/>
+      </geometry>
+    </visual>
+    <inertial>
+      <origin xyz="0 0 0" rpy="0 0 0"/>
+      <mass value="0.15"/>
+      <inertia
+        ixx=".1" ixy="0.0" ixz="0.0"
+        iyy=".1" iyz="0.0"
+        izz=".1"/>
+    </inertial>
+  </link>
+    <!-- JOINT caster_box_back TO base_link-->
+  <joint name="base_caster_box_back_joint" type="fixed">
+  <!-- NB: Z goes to - as we are below bottom deck(base)-->
+    <origin rpy="0 0 0" xyz="-${caster_X_offset_from_base_link+caster_box_lenght/2} 0 -${caster_box_height/2+base_height/2}"/>
+    <parent link="base_link"/>
+    <child link="caster_box_back"/>
+  </joint>
+     <!--*****************************-->
+    <link name="caster_sphere_back">
+    <collision name="collision">
+      <origin xyz="0 0 0" rpy="0 0 0"/>
+      <geometry>
+        <sphere radius="${caster_sphere_radius}"/>
+      </geometry>
+    </collision>
+    <visual name="caster_sphere_back_visual">
+      <origin xyz="0 0 0" rpy="0 0 0"/>
+      <geometry>
+        <sphere radius="${caster_sphere_radius}"/>
+      </geometry>
+    </visual>
+    <inertial>
+      <origin xyz="0 0 0" rpy="0 0 0"/>
+      <mass value="0.15"/>
+      <inertia
+        ixx=".1" ixy="0.0" ixz="0.0"
+        iyy=".1" iyz="0.0"
+        izz=".1"/>
+    </inertial>
+  </link>
+    <!-- JOINT caster_sphere_back TO caster_box_back-->
+  <joint name="caster_box_back_caster_sphere_back_joint" type="fixed">
+  <!-- NB: Z goes to - as we are below bottom deck(base)-->
+    <origin rpy="0 0 0" xyz="0 0 -${caster_box_lenght/2+caster_sphere_radius}"/>
+    <parent link="caster_box_back"/>
+    <child link="caster_sphere_back"/>
+  </joint>
+<!--########################################-->
+<!--######### SECOND DECK ###############################-->
+  <!-- JOINT second_deck TO BASE_LINK -->
+  <joint name="base_link_second_deck_joint" type="fixed">
+    <origin rpy="0 0 0" xyz="0 0 ${second_deck_from_base_link_Z_offset}"/>
+    <parent link="base_link"/>
+    <child link="second_deck"/>
+  </joint>
+  <!-- BASE-LINK -->
+  <!--Center on the bottom side of the base plate of the robot-->
+  <link name='second_deck'>
+    <pose>0 0 0.1 0 0 0</pose>
+    <inertial>
+      <mass value="${second_deck_mass}"/>
+      <origin xyz="0.0 0 0.1" rpy=" 0 0 0"/>
+      <inertia
+          ixx="0.1" ixy="0" ixz="0"
+          iyy="0.1" iyz="0"
+          izz="0.1"
+      />
+    </inertial>
+    <collision name='collision'>
+      <geometry>
+       <cylinder radius="${second_deck_radius}" length="${second_deck_height}"/>
+      </geometry>
+    </collision>
+    <visual name='second_deck_visual'>
+      <origin xyz="0 0 0" rpy="${M_PI_2} 0 ${M_PI_2}"/>
+      <geometry>
+        <!--<cylinder radius="${base_radius}" length="${base_height}"/>-->
+        <mesh filename="$(find robko18_description)/meshes/ArloBottomplateTST.dae" scale="0.001 0.001 0.001"/>
+      </geometry>
+      <material name="orange"/>
+    </visual>
+  </link>
+<!--########################################-->
+<!--######### third DECK ###############################-->
+  <!-- JOINT third_deck TO BASE_LINK -->
+  <joint name="third_deck_second_deck_joint" type="fixed">
+    <origin rpy="0 0 0" xyz="0 0 ${third_deck_from_base_link_Z_offset}"/>
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
Commit message: added kinect nount point and kunect deck visualisation

File: src/robko18_description/urdf/robko18.xacro (robot description, xacro)
@@ -4,4 +4,6 @@
   <xacro:include filename="$(find robko18_description)/urdf/materials.xacro" />
   <xacro:include filename="$(find robko18_description)/urdf/macros.xacro" />
+  <!-- 3D Sensors -->
+  <!--<xacro:include filename="$(find robko18_description)/urdf/kinect.urdf.xacro"/>-->
   <!-- ####### generic constants ##### -->
   <!--All units in m-kg-s-radians unit system -->
@@ -31,13 +33,20 @@
   <xacro:property name="BASE_PLATE_FROM_BASE_FRAME_Z_OFFSET" value="${0.10+(base_height/2)}" /> <!-- meters -->
  <!-- second_deck - Base Plate/Deck Cylinder base   -->
-  <xacro:property name="second_deck_from_base_link_Z_offset" value="0.145"/>
+  <xacro:property name="second_deck_from_base_link_Z_offset" value="${0.145+(second_deck_height/2)}"/>
   <xacro:property name="second_deck_height" value="${0.375*SCALE_in_m}" />
   <xacro:property name="second_deck_radius" value="${17.75*SCALE_in_m}" />
   <xacro:property name="second_deck_mass" value="1.5" />   <!-- in kg -->
   <!-- third_deck - Base Plate/Deck Cylinder base   -->
-  <xacro:property name="third_deck_from_base_link_Z_offset" value="0.145"/>
+  <xacro:property name="third_deck_from_second_deck_Z_offset" value="${0.156+(third_deck_height/2)}"/>
   <xacro:property name="third_deck_height" value="${0.375*SCALE_in_m}" />
   <xacro:property name="third_deck_radius" value="${17.75*SCALE_in_m}" />
   <xacro:property name="third_deck_mass" value="1.5" />   <!-- in kg -->
+ <!-- kinect_mount_point - joint data for maunting kinect relative to base_link  -->
+  <xacro:property name="kinect_mount_point_from_base_link_Z_offset" value="0.90"/>
+  <xacro:property name="kinect_mount_point_from_base_link_X_offset" value="-${base_radius - 0.10}"/>
+  <xacro:property name="kinect_deck_height" value="0.02" />
+  <xacro:property name="kinect_deck_width" value="0.05" />
+  <xacro:property name="kinect_deck_lenght" value="0.05" />
+  <xacro:property name="kinect_deck_mass" value=".05" />    <!--in kg-->
   <!-- Wheels -->
   <xacro:property name="wheel_diameter" value="${6*SCALE_in_m}"/>
@@ -309,6 +318,5 @@
     <child link="second_deck"/>
   </joint>
-  <!-- BASE-LINK -->
-  <!--Center on the bottom side of the base plate of the robot-->
+  <!--Centered on the bottom side of the second deck/plate of the robot-->
   <link name='second_deck'>
     <pose>0 0 0.1 0 0 0</pose>
@@ -337,12 +345,11 @@
   </link>
 <!--########################################-->
-<!--######### third DECK ###############################-->
-  <!-- JOINT third_deck TO BASE_LINK -->
+<!--######### THIRD DECK ###############################-->
+  <!-- JOINT THIRD_DECK TO SECOND_DECK -->
   <joint name="third_deck_second_deck_joint" type="fixed">
-    <origin rpy="0 0 0" xyz="0 0 ${third_deck_from_base_link_Z_offset}"/>
+    <origin rpy="0 0 0" xyz="0 0 ${third_deck_from_second_deck_Z_offset}"/>
     <parent link="second_deck"/>
     <child link="third_deck"/>
   </joint>
-  <!-- BASE-LINK -->
   <!--Center on the bottom side of the base plate of the robot-->
   <link name='third_deck'>
@@ -372,5 +379,39 @@
   </link>
 <!--########################################-->
-  <link name="camera">
+<!--######### KINECT DECK ###############################-->
+  <!-- JOINT THIRD_DECK TO SECOND_DECK -->
+  <joint name="Kinect_deck_to_base_link_joint" type="fixed">
+    <origin rpy="0 0 0" xyz="${kinect_mount_point_from_base_link_X_offset} 0 ${kinect_mount_point_from_base_link_Z_offset}"/>
+    <parent link="base_link"/>
+    <child link="kinect_deck"/>
+  </joint>
+  <!--Center on the bottom side of the base plate of the robot-->
+  <link name='kinect_deck'>
+    <pose>0 0 0.1 0 0 0</pose>
+    <inertial>
+      <mass value="${kinect_deck_mass}"/>
+      <origin xyz="0.0 0 0.1" rpy=" 0 0 0"/>
+      <inertia
+          ixx="0.1" ixy="0" ixz="0"
+          iyy="0.1" iyz="0"
+          izz="0.1"
+      />
+    </inertial>
+    <collision name='collision'>
+      <geometry>
+        <box size="${kinect_deck_width} ${kinect_deck_height} ${kinect_deck_lenght}" />
+      </geometry>
+    </collision>
+    <visual name='third_deck__visual'>
+      <origin xyz="0 0 0" rpy="0 0 0"/>
+      <geometry>
+        <box size="${kinect_deck_width} ${kinect_deck_height} ${kinect_deck_lenght}" />
+      </geometry>
+      <material name="red"/>
+    </visual>
+  </link>
+<!--########################################-->
+<!--############# CAMERA ###########################-->
+  <!--<link name="camera">
     <collision>
       <origin xyz="0 0 0" rpy="0 0 0"/>
@@ -398,5 +439,7 @@
     <parent link="base_link"/>
     <child link="camera"/>
-  </joint>
+  </joint>-->
+<!--##############################################-->
+<!--############### HOUYO LASER ##################-->
   <joint name="hokuyo_joint" type="fixed">
     <axis xyz="0 1 0" />
