Commit message: add kinect-support deck

File: src/robko18_description/urdf/robko18.xacro (robot description, xacro)
@@ -1,3 +1,3 @@
-<?xml version='1.0'?>
+<?xml version="1.0"?>
 <robot name="robko18" xmlns:xacro="http://www.ros.org/wiki/xacro">
   <xacro:include filename="$(find robko18_description)/urdf/robko18.gazebo" />
@@ -27,5 +27,5 @@
   <xacro:property name="base_from_base_frame_Z_offset" value="0.10"/>
   <xacro:property name="base_height" value="${0.375*SCALE_in_m}" />
-  <xacro:property name="base_radius" value="${17.75*SCALE_in_m}" />
+  <xacro:property name="base_radius" value="${17.75*SCALE_in_m/2}" />
   <!-- in kg weight with the battery holder plate bellow -->
   <xacro:property name="base_mass" value="1.75" />
@@ -35,18 +35,19 @@
   <xacro:property name="second_deck_from_base_link_Z_offset" value="${0.145+(second_deck_height/2)}"/>
   <xacro:property name="second_deck_height" value="${0.375*SCALE_in_m}" />
-  <xacro:property name="second_deck_radius" value="${17.75*SCALE_in_m}" />
+  <xacro:property name="second_deck_radius" value="${17.75*SCALE_in_m/2}" />
   <xacro:property name="second_deck_mass" value="1.5" />   <!-- in kg -->
   <!-- third_deck - Base Plate/Deck Cylinder base   -->
   <xacro:property name="third_deck_from_second_deck_Z_offset" value="${0.156+(third_deck_height/2)}"/>
   <xacro:property name="third_deck_height" value="${0.375*SCALE_in_m}" />
-  <xacro:property name="third_deck_radius" value="${17.75*SCALE_in_m}" />
+  <xacro:property name="third_deck_radius" value="${17.75*SCALE_in_m/2}" />
   <xacro:property name="third_deck_mass" value="1.5" />   <!-- in kg -->
  <!-- kinect_mount_point - joint data for maunting kinect relative to base_link  -->
-  <xacro:property name="kinect_mount_point_from_base_link_Z_offset" value="0.90"/>
-  <xacro:property name="kinect_mount_point_from_base_link_X_offset" value="-${base_radius - 0.10}"/>
-  <xacro:property name="kinect_deck_height" value="0.02" />
-  <xacro:property name="kinect_deck_width" value="0.05" />
-  <xacro:property name="kinect_deck_lenght" value="0.05" />
-  <xacro:property name="kinect_deck_mass" value=".05" />    <!--in kg-->
+  <xacro:property name="kinect_mount_point_from_base_link_Z_offset" value="0.50"/>
+  <!--<xacro:property name="kinect_mount_point_from_base_link_X_offset" value="-${base_radius - 0.10}"/> -->
+  <xacro:property name="kinect_mount_point_from_base_link_X_offset" value="-${0.14509}"/>
+  <xacro:property name="kinect_support_height" value="0.02" />
+  <xacro:property name="kinect_support_width" value="0.01" />
+  <xacro:property name="kinect_support_lenght" value="0.02" />
+  <xacro:property name="kinect_support_mass" value=".05" />    <!--in kg-->
   <!-- Wheels -->
   <xacro:property name="wheel_diameter" value="${6*SCALE_in_m}"/>
@@ -102,5 +103,5 @@
   <!-- BASE-LINK -->
   <!--Center on the bottom side of the base plate of the robot-->
-  <link name='base_link'>
+  <link name="base_link">
     <pose>0 0 0.1 0 0 0</pose>
     <inertial>
@@ -113,10 +114,10 @@
       />
     </inertial>
-    <collision name='collision'>
+    <collision name="collision">
       <geometry>
        <cylinder radius="${base_radius}" length="${base_height}"/>
       </geometry>
     </collision>
-    <visual name='base_visual'>
+    <visual name="base_visual">
       <origin xyz="0 0 0" rpy="${M_PI_2} 0 ${M_PI_2}"/>
       <geometry>
@@ -135,7 +136,9 @@
     </collision>
     <visual name="left_wheel_visual">
-      <origin xyz="0 0 0" rpy="0 1.5707 1.5707"/>
-      <geometry>
-        <cylinder radius="${wheel_radius}" length="${wheel_width}"/>
+      <!--<origin xyz="0 0 0" rpy="0 1.5707 1.5707"/>-->
+      <origin xyz="0 0 0" rpy="0 0 1.5707"/>
+      <geometry>
+        <mesh filename="$(find robko18_description)/meshes/wheel.dae" scale="0.0012 0.0012 0.0012"/>
+        <!--<cylinder radius="${wheel_radius}" length="${wheel_width}"/>-->
       </geometry>
     </visual>
@@ -157,7 +160,9 @@
     </collision>
     <visual name="right_wheel_visual">
-      <origin xyz="0 0 0" rpy="0 1.5707 1.5707"/>
-      <geometry>
-        <cylinder radius="${wheel_radius}" length="${wheel_width}"/>
+      <!--<origin xyz="0 0 0" rpy="0 1.5707 1.5707"/>-->
+      <origin xyz="0 0 0" rpy="0 0 1.5707"/>
+      <geometry>
+        <!--<cylinder radius="${wheel_radius}" length="${wheel_width}"/>-->
+        <mesh filename="$(find robko18_description)/meshes/wheel.dae" scale="0.0012 0.0012 0.0012"/>
       </geometry>
     </visual>
@@ -319,5 +324,5 @@
   </joint>
   <!--Centered on the bottom side of the second deck/plate of the robot-->
-  <link name='second_deck'>
+  <link name="second_deck">
     <pose>0 0 0.1 0 0 0</pose>
     <inertial>
@@ -330,10 +335,10 @@
       />
     </inertial>
-    <collision name='collision'>
+    <collision name="collision">
       <geometry>
        <cylinder radius="${second_deck_radius}" length="${second_deck_height}"/>
       </geometry>
     </collision>
-    <visual name='second_deck_visual'>
+    <visual name="second_deck_visual">
       <origin xyz="0 0 0" rpy="${M_PI_2} 0 ${M_PI_2}"/>
       <geometry>
@@ -353,5 +358,5 @@
   </joint>
   <!--Center on the bottom side of the base plate of the robot-->
-  <link name='third_deck'>
+  <link name="third_deck">
     <pose>0 0 0.1 0 0 0</pose>
     <inertial>
@@ -364,10 +369,10 @@
       />
     </inertial>
-    <collision name='collision'>
+    <collision name="collision">
       <geometry>
        <cylinder radius="${third_deck_radius}" length="${third_deck_height}"/>
       </geometry>
     </collision>
-    <visual name='third_deck__visual'>
+    <visual name="third_deck__visual">
       <origin xyz="0 0 0" rpy="${M_PI_2} 0 ${M_PI_2}"/>
       <geometry>
@@ -379,16 +384,16 @@
   </link>
 <!--########################################-->
-<!--######### KINECT DECK ###############################-->
-  <!-- JOINT THIRD_DECK TO SECOND_DECK -->
-  <joint name="Kinect_deck_to_base_link_joint" type="fixed">
+<!--######### KINECT SUPPORT ###############################-->
+  <!-- JOINT KINECT_SUPPORT TO BASE_LINK -->
+  <joint name="Kinect_support_to_base_link_joint" type="fixed">
     <origin rpy="0 0 0" xyz="${kinect_mount_point_from_base_link_X_offset} 0 ${kinect_mount_point_from_base_link_Z_offset}"/>
     <parent link="base_link"/>
-    <child link="kinect_deck"/>
-  </joint>
-  <!--Center on the bottom side of the base plate of the robot-->
-  <link name='kinect_deck'>
+    <child link="kinect_support"/>
+  </joint>
+  <!--BASE LINK IS AT center on the bottom side of the base deck/plate of the robot-->
+  <link name="kinect_support">
     <pose>0 0 0.1 0 0 0</pose>
     <inertial>
-      <mass value="${kinect_deck_mass}"/>
+      <mass value="${kinect_support_mass}"/>
       <origin xyz="0.0 0 0.1" rpy=" 0 0 0"/>
       <inertia
@@ -398,13 +403,13 @@
       />
     </inertial>
-    <collision name='collision'>
-      <geometry>
-        <box size="${kinect_deck_width} ${kinect_deck_height} ${kinect_deck_lenght}" />
-      </geometry>
-    </collision>
-    <visual name='third_deck__visual'>
-      <origin xyz="0 0 0" rpy="0 0 0"/>
-      <geometry>
-        <box size="${kinect_deck_width} ${kinect_deck_height} ${kinect_deck_lenght}" />
+    <collision name="collision">
+      <geometry>
+        <box size="${kinect_support_height} ${kinect_support_lenght} ${kinect_support_width}" />
+      </geometry>
+    </collision>
+    <visual name="kinect_support__visual">
+      <origin xyz="0 0 0" rpy="0 0 0"/>
+      <geometry>
+        <box size="${kinect_support_height} ${kinect_support_lenght} ${kinect_support_width}" />
       </geometry>
       <material name="red"/>
