Commit message: kinect in gazebo, decks missing in Rviz

File: src/robko18_description/urdf/common.xacro (robot description, xacro)
@@ -1,6 +1,8 @@
 <?xml version="1.0"?>
-<robot
-  xmlns:xacro="http://ros.org/wiki/xacro">
-  <property name="M_PI" value="3.1415926535897931" />
+  <!--
+  Various useful properties such as constants and materials
+ -->
+<robot name="xacro_properties" xmlns:xacro="http://ros.org/wiki/xacro">
+  <xacro:property name="M_PI" value="3.1415926535897931" />
 <!-- generic constants -->
   <xacro:property name="M_PI" value="3.14159265359" />

File: src/robko18_description/urdf/robko18.xacro (robot description, xacro)
@@ -5,5 +5,5 @@
   <xacro:include filename="$(find robko18_description)/urdf/macros.xacro" />
   <!-- 3D Sensors -->
-  <!--<xacro:include filename="$(find robko18_description)/urdf/kinect.urdf.xacro"/>-->
+  <xacro:include filename="$(find robko18_description)/urdf/kinect.urdf.xacro"/>
   <!-- ####### generic constants ##### -->
   <!--All units in m-kg-s-radians unit system -->
@@ -23,5 +23,5 @@
 Weight = 3.5 lbs (1.59 kg) per assembly
 Dimensions: 17.375 inches (44.13 cm) diameter x .375 inches (.95 cm) thick
--->  second_deck
+-->
   <!-- base_link - Base Plate/Deck Cylinder base   -->
   <xacro:property name="base_from_base_frame_Z_offset" value="0.10"/>
@@ -473,3 +473,4 @@
     </inertial>
   </link>
+   <sensor_kinect  parent="kinect_support"/>
 </robot>
