Commit message: changed find package to direct path - now model shows correctly in rviz

File: src/robko18_description/urdf/kinect.urdf.xacro (robot description, xacro)
@@ -27,5 +27,6 @@
        <origin xyz="0 0 0" rpy="0 0 ${M_PI/2}"/>
         <geometry>
-          <mesh filename="$(find robko18_description)/meshes/kinect.dae"/>
+          <mesh filename="package://robko18_description/meshes/kinect.dae"/>
+          <!--<mesh filename="$(find robko18_description)/meshes/kinect.dae"/>          -->
          <!--<mesh filename="package://turtlebot_description/meshes/sensors/kinect.dae"/>-->
         </geometry>

File: src/robko18_description/urdf/robko18_test.urdf.xacro (robot description, xacro)
@@ -1,9 +1,9 @@
 <?xml version="1.0"?>
 <robot name="robko18" xmlns:xacro="http://www.ros.org/wiki/xacro">
-  <xacro:include filename="$(find robko18_description)/urdf/robko18.gazebo" />
+  <xacro:include filename="$(find robko18_description)/urdf/robko18_gazebo.urdf.xacro" />
   <xacro:include filename="$(find robko18_description)/urdf/materials.xacro" />
   <xacro:include filename="$(find robko18_description)/urdf/macros.xacro" />
   <!-- 3D Sensors -->
-  <xacro:include filename="$(find robko18_description)/urdf/kinect.urdf.xacro"/>
+  <!--<xacro:include filename="$(find robko18_description)/urdf/kinect.urdf.xacro"/>-->
   <!-- ####### generic constants ##### -->
   <!--All units in m-kg-s-radians unit system -->
@@ -122,7 +122,6 @@
       <origin xyz="0 0 0" rpy="${M_PI_2} 0 ${M_PI_2}"/>
       <geometry>
-        <!--<cylinder radius="${base_radius}" length="${base_height}"/>-->
+        <cylinder radius="${base_radius}" length="${base_height}"/>
         <!--<mesh filename="$(find robko18_description)/meshes/ArloBottomplateTST.dae" scale="0.001 0.001 0.001"/>-->
-        <mesh filename="package://robko18_description/meshes/ArloBottomplateTST.dae" scale="0.001 0.001 0.001"/>
       </geometry>
       <material name="orange"/>
@@ -141,6 +140,5 @@
       <geometry>
         <!--<mesh filename="$(find robko18_description)/meshes/wheel.dae" scale="0.0012 0.0012 0.0012"/>-->
-        <mesh filename="package://robko18_description/meshes/wheel.dae" scale="0.0012 0.0012 0.0012"/>
-        <!--<cylinder radius="${wheel_radius}" length="${wheel_width}"/>-->
+        <cylinder radius="${wheel_radius}" length="${wheel_width}"/>
       </geometry>
     </visual>
@@ -165,7 +163,6 @@
       <origin xyz="0 0 0" rpy="0 0 1.5707"/>
       <geometry>
-        <!--<cylinder radius="${wheel_radius}" length="${wheel_width}"/>-->
+        <cylinder radius="${wheel_radius}" length="${wheel_width}"/>
         <!--<mesh filename="$(find robko18_description)/meshes/wheel.dae" scale="0.0012 0.0012 0.0012"/>-->
-        <mesh filename="package://robko18_description/meshes/wheel.dae" scale="0.0012 0.0012 0.0012"/>
       </geometry>
     </visual>
@@ -346,7 +343,6 @@
       <origin xyz="0 0 0" rpy="${M_PI_2} 0 ${M_PI_2}"/>
       <geometry>
-        <!--<cylinder radius="${base_radius}" length="${base_height}"/>-->
+        <cylinder radius="${base_radius}" length="${base_height}"/>
         <!--<mesh filename="$(find robko18_description)/meshes/ArloBottomplateTST.dae" scale="0.001 0.001 0.001"/>-->
-        <mesh filename="package://robko18_description/meshes/ArloBottomplateTST.dae" scale="0.001 0.001 0.001"/>
       </geometry>
       <material name="orange"/>
@@ -423,5 +419,5 @@
 <!--########################################-->
 <!--############# CAMERA ###########################-->
-  <!--<link name="camera">
+  <link name="camera">
     <collision>
       <origin xyz="0 0 0" rpy="0 0 0"/>
@@ -449,5 +445,5 @@
     <parent link="base_link"/>
     <child link="camera"/>
-  </joint>-->
+  </joint>
 <!--##############################################-->
 <!--############### HOUYO LASER ##################-->
@@ -478,6 +474,6 @@
     </inertial>
   </link>
-  <xacro:include filename="$(find robko18_description)/urdf/robko18_gazebo.urdf.xacro"/>
+  <!--<xacro:include filename="$(find robko18_description)/urdf/robko18_gazebo.urdf.xacro"/>
   <xacro:include filename="$(find robko18_description)/urdf/robko18_properties.urdf.xacro"/>
-   <sensor_kinect  parent="kinect_support"/>
+   <sensor_kinect  parent="kinect_support"/>-->
 </robot>
