Commit message: add CPRMover4 urdf and meshes, attac arm to robot

File: src/robko18_description/urdf/robko18_mover4.urdf.xacro (robot description, xacro)
@@ -502,7 +502,11 @@
   <!-- JOINT  arm_maunt_point TO BASE_LINK -->
   <joint name="base_footprint_arm_maunt_point_joint" type="fixed">
-    <origin rpy="0 0 0" xyz="${arm_mount_point_from_base_frame_X_offset} 0 ${arm_mount_point_from_base_frame_Z_offset}"/>
+    <!--<origin rpy="0 0 0" xyz="map_bf_X_offset 0 amp_bf_Z_offset"/>-->
+        <!--<origin rpy="0 0 0" xyz="0.15 0 0.4"/>-->
+        <origin rpy="0 0 0" xyz="${arm_mount_point_from_base_frame_X_offset} 0 ${arm_mount_point_from_base_frame_Z_offset}"/>
     <parent link="base_footprint"/>
     <child link="arm_maunt_point"/>
   </joint>
+   <xacro:include filename="$(find robko18_description)/urdf/CPRMover4.urdf.xacro" />
+<xacro:CPRMover4_arm name="mover4_arm" parent="arm_maunt_point"/>
 </robot>
