Commit message: working on cprmover4 simulation

File: src/robko18_description/urdf/cprmover4_standalone.urdf.xacro (robot description, xacro)
@@ -1,48 +1,8 @@
 <?xml version="1.0"?>
-<robot name="robot_description" xmlns:xacro="http://www.ros.org/wiki/xacro">
- <!-- base_link - Base Plate/Deck Cylinder base   -->
-   <xacro:property name="wheel_diameter" value="${6*SCALE_in_m}"/>
-  <xacro:property name="wheel_radius" value="${wheel_diameter/2}"/>
-  <xacro:property name="wheel_width" value="0.03"/><!--set to tyre width-->
-  <xacro:property name="wheel_mass" value="0.6" /> --> <!-- ???? in kg-->
-  <xacro:property name="base_from_base_frame_Z_offset" value="0.10"/>
-  <xacro:property name="base_height" value="${0.375*SCALE_in_m}" />
-  <xacro:property name="base_radius" value="${17.75*SCALE_in_m/2}" />
-    <xacro:property name="BASE_PLATE_FROM_BASE_FRAME_Z_OFFSET" value="${0.10+(base_height/2)}" /> <!-- meters -->
-  <!-- in kg weight with the battery holder plate bellow -->
-  <xacro:property name="base_mass" value="1.75" />
-  <xacro:property name="M_PI" value="3.1415926535897931" />
-  <xacro:property name="M_PI_2" value="1.570796327" />
-  <xacro:property name="DEG_TO_RAD" value="0.017453293" />
-  <xacro:property name="SCALE_in_m" value="0.0254"/> <!--inches to meters-->
-  <xacro:property name="SCALE_mm_m" value="0.001"/> <!--milimeters to meters-->
-  <xacro:property name="base_x_origin_to_wheel_origin" value="0.0" />
-  <xacro:property name="base_y_origin_to_wheel_origin" value="0.2" />
-    <!--<xacro:property name="base_y_origin_to_wheel_origin" value="0.19" />-->
-  <xacro:property name="base_z_origin_to_wheel_origin" value="${BASE_PLATE_FROM_BASE_FRAME_Z_OFFSET - wheel_radius}" />
+<robot name="cprmover4" xmlns:xacro="http://ros.org/wiki/xacro" >
+<!--<robot xmlns:xacro="http://ros.org/wiki/xacro" >-->
 <!-- URDF file for the Commonplace Robotics Mover4 robot arm -->
 <!-- Version 1.1 from Oct. 04th, 2016. -->
-  <link name="base_footprint">
-    <inertial>
-      <mass value="5"/>
-      <origin xyz="0 0 0"/>
-      <inertia ixx="0.0001" ixy="0.0" ixz="0.0" iyy="0.0001" iyz="0.0" izz="0.0001"/>
-    </inertial>
-    <visual>
-      <origin rpy="0 0 0" xyz="0 0 0"/>
-      <geometry>
-        <box size="0.001 0.001 0.001"/>
-      </geometry>
-      <material name="red"/>
-    </visual>
-  </link>
-  <gazebo reference="base_footprint">
-    <turnGravityOff>false</turnGravityOff>
-  </gazebo>
-  <!-- JOINT BASE_LINK TO BASE_FRAME-->
-  <joint name="base_footprint_base_link_joint" type="fixed">
-    <origin rpy="0 0 0" xyz="0 0 0.10"/>
-    <parent link="base_footprint"/>
-    <child link="base_link"/>
+<!--<xacro:macro name="CPRMover4_arm" params="parent name *origin">-->
 <link name="base_link">
 <pose>0 0 0.1 0 0 0</pose>

File: src/robko18_description/urdf/cprmover4_standalone_sim.urdf.xacro (robot description, xacro)
@@ -1,32 +1,9 @@
 <?xml version="1.0"?>
-<robot name="robot_description" xmlns:xacro="http://www.ros.org/wiki/xacro">
- <!-- base_link - Base Plate/Deck Cylinder base   -->
-   <xacro:property name="wheel_diameter" value="${6*SCALE_in_m}"/>
-  <xacro:property name="wheel_radius" value="${wheel_diameter/2}"/>
-  <xacro:property name="wheel_width" value="0.03"/><!--set to tyre width-->
-  <xacro:property name="wheel_mass" value="0.6" /> --> <!-- ???? in kg-->
-  <xacro:property name="base_from_base_frame_Z_offset" value="0.10"/>
-  <xacro:property name="base_height" value="${0.375*SCALE_in_m}" />
-  <xacro:property name="base_radius" value="${17.75*SCALE_in_m/2}" />
-    <xacro:property name="BASE_PLATE_FROM_BASE_FRAME_Z_OFFSET" value="${0.10+(base_height/2)}" /> <!-- meters -->
-  <!-- in kg weight with the battery holder plate bellow -->
-  <xacro:property name="base_mass" value="1.75" />
-  <xacro:property name="M_PI" value="3.1415926535897931" />
-  <xacro:property name="M_PI_2" value="1.570796327" />
-  <xacro:property name="DEG_TO_RAD" value="0.017453293" />
-  <xacro:property name="SCALE_in_m" value="0.0254"/> <!--inches to meters-->
-  <xacro:property name="SCALE_mm_m" value="0.001"/> <!--milimeters to meters-->
-  <xacro:property name="base_x_origin_to_wheel_origin" value="0.0" />
-  <xacro:property name="base_y_origin_to_wheel_origin" value="0.2" />
-    <!--<xacro:property name="base_y_origin_to_wheel_origin" value="0.19" />-->
-  <xacro:property name="base_z_origin_to_wheel_origin" value="${BASE_PLATE_FROM_BASE_FRAME_Z_OFFSET - wheel_radius}" />
+<robot name="cprmover4" xmlns:xacro="http://ros.org/wiki/xacro" >
+<!--<robot xmlns:xacro="http://ros.org/wiki/xacro" >-->
 <!-- URDF file for the Commonplace Robotics Mover4 robot arm -->
 <!-- Version 1.1 from Oct. 04th, 2016. -->
+<!--<xacro:macro name="CPRMover4_arm" params="parent name *origin">-->
   <link name="base_footprint">
-    <inertial>
-      <mass value="5"/>
-      <origin xyz="0 0 0"/>
-      <inertia ixx="0.0001" ixy="0.0" ixz="0.0" iyy="0.0001" iyz="0.0" izz="0.0001"/>
-    </inertial>
     <visual>
       <origin rpy="0 0 0" xyz="0 0 0"/>
@@ -42,14 +19,15 @@
   <!-- JOINT BASE_LINK TO BASE_FRAME-->
   <joint name="base_footprint_base_link_joint" type="fixed">
-    <origin rpy="0 0 0" xyz="0 0 0.10"/>
+    <origin rpy="0 0 0" xyz="0 0 0"/>
     <parent link="base_footprint"/>
     <child link="base_link"/>
+  </joint>
 <link name="base_link">
-<pose>0 0 0.1 0 0 0</pose>
-    <inertial>
+<!--<pose>0 0 0.1 0 0 0</pose>-->
+    <!--<inertial>
       <mass value="0.5"/>
       <origin xyz="0 0 0"/>
       <inertia ixx="0.0001" ixy="0.0" ixz="0.0" iyy="0.0001" iyz="0.0" izz="0.0001"/>
-    </inertial>
+    </inertial>-->
     <visual>
 	<origin rpy="0 0 0" xyz="0 0 0.0"/>
@@ -275,3 +253,34 @@
     <joint_properties damping="0.0" friction="0.0"/>
   </joint>
+<!-- Transmissions macro    -->
+<xacro:macro name="transmission_block" params="joint_name">
+	  <transmission name="tran_${joint_name}">
+	    <type>transmission_interface/SimpleTransmission</type>
+	    <joint name="${joint_name}">
+	      <hardwareInterface>PositionJointInterface</hardwareInterface>
+	    </joint>
+	    <actuator name="motor_${joint_name}">
+	      <hardwareInterface>PositionJointInterface</hardwareInterface>
+	      <mechanicalReduction>1</mechanicalReduction>
+	    </actuator>
+	  </transmission>
+   </xacro:macro>
+    <!-- Transmissions for ROS Control -->
+   <xacro:transmission_block joint_name="Joint0"/>
+   <xacro:transmission_block joint_name="Joint1"/>
+   <xacro:transmission_block joint_name="Joint2"/>
+   <xacro:transmission_block joint_name="Joint3"/>
+   <xacro:transmission_block joint_name="Gripper1"/>
+   <xacro:transmission_block joint_name="Gripper2"/>
+     <!-- ros_control plugin -->
+<!--<gazebo>
+  <plugin name="gazebo_ros_control" filename="libgazebo_ros_control.so">
+    <robotNamespace>/cprmover4</robotNamespace>
+  </plugin>
+</gazebo>-->
+<gazebo>
+  <plugin name="gazebo_ros_control" filename="libgazebo_ros_control.so">
+    <robotNamespace>/cprmover4</robotNamespace>
+  </plugin>
+</gazebo>
 </robot>
